Commit message: Rotate visual and collision origins by 1.57 radians

File: bebop_gazebo/urdf/bebop_base.urdf.xacro (robot description, xacro)
@@ -21,5 +21,5 @@
       </inertial>
       <visual>
-        <origin xyz="0 0 0" rpy="0 0 0" />
+        <origin xyz="0 0 0" rpy="0 0 1.57" />
         <geometry>
           <mesh filename="package://bebop_gazebo/meshes/bebop_model.stl"/>
@@ -30,5 +30,5 @@
       </visual>
       <collision>
-        <origin xyz="0 0 0" rpy="0 0 0" />
+        <origin xyz="0 0 0" rpy="0 0 1.57" />
         <geometry>
           <mesh filename="package://bebop_gazebo/meshes/bebop_model.stl"/>

Commit message: Update bebop_base.urdf.xacro

File: bebop_gazebo/urdf/bebop_base.urdf.xacro (robot description, xacro)
@@ -41,5 +41,5 @@
     <link name="camera_optical"></link>
     <joint name="base_link_joint" type="fixed">
-      <origin xyz="${camera_offset_len} 0 ${camera_offset_ver}" rpy="0 0 0" />
+      <origin xyz="0 ${camera_offset_len} ${camera_offset_ver}" rpy="0 0 1.57" />
       <parent link="base_link"/>
       <child link="camera_base_link" />
@@ -63,4 +63,5 @@
     <joint name="camera_optical_joint" type="fixed">
       <origin xyz="0 0 0" rpy="${-pi/2} 0 ${-pi/2}" />
+      <!-- <origin xyz="0 0 0" rpy="0 0 0" /> -->
       <parent link="camera_tilt_link" />
       <child link="camera_optical" />

Commit message: Change material color from blue to black in URDF

File: bebop_gazebo/urdf/bebop_base.urdf.xacro (robot description, xacro)
@@ -25,6 +25,6 @@
           <mesh filename="package://bebop_gazebo/meshes/bebop_model.stl"/>
         </geometry>
-        <material name="blue">
-          <color rgba="0 0.4 0.6 1"/>
+        <material name="black">
+          <color rgba="0 0 0 1"/>
         </material>
       </visual>
@@ -36,4 +36,7 @@
       </collision>
     </link>
+    <gazebo reference="base_link">
+      <material>Gazebo/Black</material>
+    </gazebo>
     <link name="camera_base_link"></link>
     <link name="camera_pan_link"></link>
